File: armbian/kicad/remoteControl/kicad/remoteControl.kicad_pcb (KiCad board)
At the start: 2 copper layers, 162.6 x 101.6 mm, 28 parts, among them J1 Conn_01x02, J2 USB_2, P1 CONN_1, P10 CONN_2, P11 CONN_1, P12 CONN_1, P13 CONN_1, P14 CONN_3, P16 CONN_1, P17 CONN_1, P2 CONN_1, P3 PI, P4 CONN_5, P5 CONN_4X1, P6 CONN_3, P7 CONN_4X1, P8 CONN_2, P9 CONN_2, U1 BUCK

Commit message: armbian/kicad/remoteControl pcb (5)
Parts:
- added P15: CONN_1, kicad:PIN_ARRAY_1X1, F.Cu at (182.9, 121.9)
- added P18: CONN_1, kicad:PIN_ARRAY_1X1, F.Cu at (185.4, 121.9)
- added P19: CONN_1, kicad:PIN_ARRAY_1X1, F.Cu at (188.0, 121.9)
- P5: value CONN_4X1 -> CONN_1; footprint kicad:PIN_ARRAY_4X1 -> kicad:PIN_ARRAY_1X1
- moved P5 3.81 mm to (180.3, 121.9), turned to 0 degrees
Connections:
- P3 pad 1: Net-(P3-Pad1) -> Net-(P19-Pad1)
- P3 pad 10: (no net) -> Net-(P3-Pad10)
- P3 pad 11: Net-(P3-Pad11) -> Net-(P15-Pad1)
- P3 pad 12: (no net) -> Net-(P3-Pad12)
- P3 pad 14: (no net) -> Net-(P3-Pad14)
- P3 pad 16: (no net) -> Net-(P3-Pad16)
- P3 pad 18: (no net) -> Net-(P3-Pad18)
- P3 pad 2: (no net) -> Net-(P3-Pad2)
- P3 pad 20: (no net) -> Net-(P3-Pad20)
- P3 pad 22: (no net) -> Net-(P3-Pad22)
- P3 pad 24: (no net) -> Net-(P3-Pad24)
- P3 pad 8: (no net) -> Net-(P3-Pad8)
- P5 pad 1: Net-(P3-Pad1) -> Net-(P3-Pad13)
- P6 pad 1: Net-(P3-Pad1) -> Net-(P19-Pad1)
- P7 pad 2: Net-(P3-Pad1) -> Net-(P19-Pad1)
- R1 pad 2: Net-(P3-Pad1) -> Net-(P19-Pad1)
Routing:
- net Net-(P3-Pad1): track 299.4 -> 0.00 mm
- net Net-(P19-Pad1): track 0.00 -> 299.4 mm
- net Net-(P3-Pad11): track 74.0 -> 0.00 mm
- net Net-(P15-Pad1): track 0.00 -> 74.0 mm
Other:
- net class Default: trace_width 0.25 -> 0.8
