File: cicd/mps/kicad/remoteControl.kicad_pcb (KiCad board)
At the start: 2 copper layers, 162.6 x 101.6 mm, 31 parts, among them J1 Conn_01x02, J2 USB_2, P1 CONN_1, P10 CONN_2, P11 CONN_1, P12 CONN_1, P13 CONN_1, P14 CONN_3, P15 CONN_1, P16 CONN_1, P17 CONN_1, P18 CONN_1, P19 CONN_1, P2 CONN_1, P3 PI, P4 CONN_5, P5 CONN_1, P6 CONN_3, P7 CONN_4X1, P8 CONN_2, P9 CONN_2, U1 BUCK

Commit message: mps/kicad: frees up the SPI pins
Parts:
- moved P17 89.2 mm to (182.9, 121.9)
- moved P15 89.0 mm to (177.8, 33.0)
- moved C2 2.54 mm to (129.5, 45.7)
- moved P16 2.54 mm to (175.3, 33.0)
Connections:
- J1 pad 1: Net-(J1-Pad1) -> Net-(J1-Pin_1)
- J1 pad 2: Net-(J1-Pad2) -> Net-(J1-Pin_2)
- P14 pad 1: Net-(J1-Pad2) -> Net-(J1-Pin_2)
- P14 pad 2: Net-(J1-Pad1) -> Net-(J1-Pin_1)
- P15 pad 1: Net-(P15-Pad1) -> Net-(J1-Pin_1)
- P16 pad 1: Net-(J1-Pad1) -> Net-(J1-Pin_2)
- P17 pad 1: Net-(J1-Pad2) -> Net-(P17-Pad1)
- P3 pad 10: Net-(P3-Pad10) -> unconnected-(P3-RX0-Pad10)
- P3 pad 11: Net-(P15-Pad1) -> Net-(P17-Pad1)
- P3 pad 12: Net-(P3-Pad12) -> Net-(P4-P3)
- P3 pad 14: Net-(P3-Pad14) -> unconnected-(P3-GND-Pad14)
- P3 pad 16: Net-(P3-Pad16) -> Net-(P4-P4)
- P3 pad 18: Net-(P3-Pad18) -> Net-(P4-P5)
- P3 pad 19: Net-(P3-Pad19) -> unconnected-(P3-MOSI-Pad19)
- P3 pad 2: Net-(P3-Pad2) -> unconnected-(P3-5V-Pad2)
- P3 pad 21: Net-(P3-Pad21) -> unconnected-(P3-MISO-Pad21)
- P3 pad 22: Net-(P3-Pad22) -> unconnected-(P3-Pad22)
- P3 pad 23: Net-(P3-Pad23) -> unconnected-(P3-SCLK-Pad23)
- P3 pad 24: Net-(P3-Pad24) -> unconnected-(P3-CS-Pad24)
- P3 pad 8: Net-(P3-Pad8) -> unconnected-(P3-TX0-Pad8)
- P4 pad 3: Net-(P3-Pad23) -> Net-(P4-P3)
- P4 pad 4: Net-(P3-Pad21) -> Net-(P4-P4)
- P4 pad 5: Net-(P3-Pad19) -> Net-(P4-P5)
- U1 pad 1: Net-(J1-Pad1) -> Net-(J1-Pin_1)
- U1 pad 2: Net-(J1-Pad2) -> Net-(J1-Pin_2)
Routing:
- net Net-(J1-Pin_1): track 0.00 -> 246.3 mm
- net Net-(J1-Pad1): track 246.3 -> 0.00 mm
- net Net-(J1-Pin_2): track 0.00 -> 230.5 mm
- net Net-(J1-Pad2): track 230.5 -> 0.00 mm
- net Net-(P4-P3): track 0.00 -> 90.7 mm
- net Net-(P3-Pad19): track 87.6 -> 0.00 mm
- net Net-(P3-Pad21): track 86.1 -> 0.00 mm
- net Net-(P3-Pad23): track 84.6 -> 0.00 mm
- net Net-(P4-P4): track 0.00 -> 83.6 mm
- net Net-(P4-P5): track 0.00 -> 78.9 mm
- net Net-(P17-Pad1): track 0.00 -> 74.0 mm
- net Net-(P15-Pad1): track 74.0 -> 0.00 mm
- net Net-(P4-P1): track 104.9 -> 93.7 mm
- net Net-(P14-P3): track 113.6 -> 111.5 mm
- net Net-(U1-OUT+): track 217.7 -> 216.3 mm
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
Commit message: mps: update kicad files for pigpio-spi
Connections:
- P3 pad 15: Net-(P14-P3) -> unconnected-(P3-Pad15)
- P3 pad 19: unconnected-(P3-MOSI-Pad19) -> Net-(P14-P3)
Routing:
- net Net-(P14-P3): track 111.5 -> 106.4 mm
Changed lines of the file:
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@@
 	(net 23 "unconnected-(P3-TX0-Pad8)")
 	(net 24 "unconnected-(P3-SCLK-Pad23)")
-	(net 25 "unconnected-(P3-MOSI-Pad19)")
+	(net 25 "unconnected-(P3-Pad15)")
 	(net 26 "unconnected-(P3-Pad22)")
 	(net 27 "unconnected-(P3-GND-Pad14)")
@@
 			(size 1.99898 1.99898)
 			(layers "F.Paste")
-			(pinfunction "GND")
-			(pintype "passive+no_connect")
 		)
 		(pad "1" thru_hole rect
@@
 			(layers "*.Cu" "*.Mask" "F.SilkS")
 			(remove_unused_layers no)
-			(net 16 "Net-(P14-P3)")
-			(pintype "passive")
+			(net 25 "unconnected-(P3-Pad15)")
+			(pintype "passive+no_connect")
 		)
 		(pad "16" thru_hole circle
@@
 			(layers "*.Cu" "*.Mask" "F.SilkS")
 			(remove_unused_layers no)
-			(net 25 "unconnected-(P3-MOSI-Pad19)")
+			(net 16 "Net-(P14-P3)")
 			(pinfunction "MOSI")
-			(pintype "passive+no_connect")
+			(pintype "passive")
 		)
 		(pad "21" thru_hole circle
@@
 		(layer "Edge.Cuts")
 	)
-	(gr_line
-		(start 109.22 22.86)
-		(end 109.22 22.86)
-		(stroke
-			(width 0.000001)
-			(type solid)
-		)
-		(layer "Edge.Cuts")
-	)
 	(gr_circle
 		(center 173.99 59.69)
@@
 	)
 	(segment
-		(start 132.08 121.92)
-		(end 68.58 121.92)
+		(start 139.7 86.36)
+		(end 144.78 91.44)
 		(width 0.8)
 		(layer "B.Cu")
@@
 	)
 	(segment
-		(start 139.7 81.28)
-		(end 144.78 86.36)
+		(start 144.78 109.22)
+		(end 132.08 121.92)
 		(width 0.8)
 		(layer "B.Cu")
@@
 	)
 	(segment
-		(start 144.78 86.36)
-		(end 144.78 109.22)
+		(start 132.08 121.92)
+		(end 68.58 121.92)
 		(width 0.8)
 		(layer "B.Cu")
@@
 	)
 	(segment
-		(start 144.78 109.22)
-		(end 132.08 121.92)
+		(start 144.78 91.44)
+		(end 144.78 109.22)
 		(width 0.8)
 		(layer "B.Cu")
